File: PCB/rgb_led_controller.kicad_pcb (KiCad board)
At the start: 2 copper layers, 68.8 x 56.9 mm, 12 parts, among them J1 Conn_01x04, J2 Conn_01x05, U1 MOUDLE-SEEEDUINO-XIAO

Commit message: Added complete Fusion 360 case - top plate and bottom case with branding
Parts:
- Mode: renamed from Color Control
- renumbered Brightness to Presets
Changed lines of the file:
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@@
 		(tenting front back)
 		(pcbplotparams
-			(layerselection 0x00000000_00000000_5555555d_5755f5ff)
+			(layerselection 0x00000000_00000000_55555555_57555550)
 			(plot_on_all_layers_selection 0x00000000_00000000_00000000_00000000)
 			(disableapertmacros no)
@@
 			(crossoutdnponfab yes)
 			(subtractmaskfromsilk no)
-			(outputformat 1)
+			(outputformat 3)
 			(mirror no)
 			(drillshape 0)
@@
 		(descr "Generic 6mm SW tactile push button")
 		(tags "tact sw push 6mm")
-		(property "Reference" "Color Control"
+		(property "Reference" "Mode"
 			(at 3.35 7.45 0)
 			(layer "F.SilkS")
@@
 		(descr "Generic 6mm SW tactile push button")
 		(tags "tact sw push 6mm")
-		(property "Reference" "Brightness"
+		(property "Reference" "Presets"
 			(at 3.35 7.45 0)
 			(layer "F.SilkS")
